Commit message: Adapting for futurhand format, first pass

File: fanuc_hardware_interface/robot/crx10ia.urdf.xacro (robot description, xacro)
@@ -9,5 +9,8 @@
   <xacro:arg name="force_sensor_type" default="1"/>
   <xacro:arg name="use_mock" default="false"/>
+  <xacro:arg name="prefix" default="fanuc"/>
+  <xacro:arg name="hand_type" default="minimal"/>
   <xacro:include filename="$(find fanuc_crx_description)/urdf/crx10ia_urdf_macro.xacro"/>
+  <xacro:include filename="$(find futur_hand_description)/hands/hand_$(arg hand_type)/xacro/hand_$(arg hand_type).xacro"/>
   <xacro:if value="$(arg use_mock)">
     <xacro:include filename="$(find fanuc_hardware_interface)/config/crx_mock_ros2_control_macro.xacro"/>
@@ -17,8 +20,17 @@
   </xacro:unless>
   <link name="world"/>
-  <link name="end_effector"/>
-  <xacro:crx10ia parent="world" child="end_effector">
+  <link name="$(arg prefix)_end_effector"/>
+  <xacro:crx10ia
+    parent="world"
+    child="$(arg prefix)_end_effector"
+    prefix="$(arg prefix)_">
     <origin xyz="0 0 0" rpy="0 0 0"/>
   </xacro:crx10ia>
-  <xacro:crx_control name="crx10ia"/>
+  <xacro:hand_description
+    parent_link="$(arg prefix)_end_effector"
+    prefix="$(arg prefix)"
+  />
+  <xacro:crx_control
+    name="crx10ia"
+    prefix="$(arg prefix)_"/>
 </robot>

Commit message: flip fanuc end effector frame 90deg so hand is mounted correclty

File: fanuc_hardware_interface/robot/crx10ia.urdf.xacro (robot description, xacro)
@@ -21,11 +21,18 @@
   <xacro:include filename="$(find futur_hand_description)/config/hand_ros2_control.xacro"/>
   <link name="world"/>
+  <link name="$(arg prefix)_end_effector_fanuc"/>
   <link name="$(arg prefix)_end_effector"/>
   <xacro:crx10ia
     parent="world"
-    child="$(arg prefix)_end_effector"
+    child="$(arg prefix)_end_effector_fanuc"
     prefix="$(arg prefix)_">
     <origin xyz="0 0 0" rpy="0 0 0"/>
   </xacro:crx10ia>
+  <!-- Reorient the end-effector frame relative to the Fanuc flange -->
+  <joint name="$(arg prefix)_end_effector_joint" type="fixed">
+    <parent link="$(arg prefix)_end_effector_fanuc"/>
+    <child  link="$(arg prefix)_end_effector"/>
+    <origin xyz="0 0 0" rpy="0 ${pi/2} 0"/>
+  </joint>
   <xacro:hand_description
     parent_link="$(arg prefix)_end_effector"

Commit message: remove unnecessary virtual joint

File: fanuc_hardware_interface/robot/crx10ia.urdf.xacro (robot description, xacro)
@@ -21,18 +21,11 @@
   <xacro:include filename="$(find futur_hand_description)/config/hand_ros2_control.xacro"/>
   <link name="world"/>
-  <link name="$(arg prefix)_end_effector_fanuc"/>
   <link name="$(arg prefix)_end_effector"/>
   <xacro:crx10ia
     parent="world"
-    child="$(arg prefix)_end_effector_fanuc"
+    child="$(arg prefix)_end_effector"
     prefix="$(arg prefix)_">
     <origin xyz="0 0 0" rpy="0 0 0"/>
   </xacro:crx10ia>
-  <!-- Reorient the end-effector frame relative to the Fanuc flange -->
-  <joint name="$(arg prefix)_end_effector_joint" type="fixed">
-    <parent link="$(arg prefix)_end_effector_fanuc"/>
-    <child  link="$(arg prefix)_end_effector"/>
-    <origin xyz="0 0 0" rpy="0 ${pi/2} 0"/>
-  </joint>
   <xacro:hand_description
     parent_link="$(arg prefix)_end_effector"
